File: assignment1/SmartHome IBM project .brd (EAGLE design)
At the start: 244.9 x 102.4 mm, 16 parts, among them K1 RELAY-SPDT_LU-5-R, K2 RELAY-SPDT_LU-5-R, M1 MOTOR_HDR, P1 BATTERYGENERIC, U1 ARDUINO-UNO-R3-SHIELD

Commit message: Assignment 1
Parts:
- removed GAS1: GAS-SENSORMQ-XX-SOCKET, Tinkercad:MQ-XX-SOCKET
- removed K1, K2: RELAY-SPDT_LU-5-R, Tinkercad:LU-5-R
- removed L1, L2: LIGHTBULB, Tinkercad:1X02
- removed M1: MOTOR_HDR, Tinkercad:MOTOR
- removed P1: BATTERYGENERIC, Tinkercad:BATTERY-GENERIC
- removed PING1: DISTANCE-SENSOR-3PIN, Tinkercad:28015
- removed S1: TOGGLE, Tinkercad:SWITCH-SPDT-PTH-8.5X3.7MM
- removed SERVO1: SERVOSG90, Tinkercad:SG90
- added D1, D2: RED, Tinkercad:LEDRD254W60D565H860B
- added R4, R5: 100, Tinkercad:RESAD1016W63L850D250B
- R2: value 1k -> 10k
- R3: value 5k -> 100
- moved R3 117.3 mm to (100.7, 21.6), turned to 360 degrees
- moved PIEZO1 109.4 mm to (126.1, 33.0), turned to -90 degrees
- moved R1 39.0 mm to (79.1, 24.1)
- moved R2 38.5 mm to (85.4, 21.6), turned to 360 degrees
- moved PIR1 8.24 mm to (82.8, 87.9)
- moved U1 3.19 mm to (29.8, 34.5)
Connections:
- removed net L1_2: L1.2, L2.2
- removed net L2_1: K2.12, L2.1
- removed net M1_+: M1.+, S1.1
- removed net M1_-: K1.6, M1.-
- removed net P1+: K2.7, P1.+, S1.2
- removed net P1-: K1.12, L1.1, P1.-
- removed net U1_A1: GAS1.1, GAS1.3, R3.1, U1.A1
- removed net U1_D10: K1.8, U1.D10
- removed net U1_D13: K2.5, U1.D13
- removed net U1_D6: PING1.3, U1.D6
- new net D1_A: D1.1, R3.2
- new net D2_A: D2.1, R4.2
- new net PIEZO1_1: PIEZO1.1, R5.2
- net U1_5V: now also R1.1; no longer GAS1.4, GAS1.5, GAS1.6, PING1.2, R2.1, SERVO1.2
- net U1_A0: now also R1.2, R2.1; no longer R1.1, R2.2
- net U1_D7: now also R3.1; no longer SERVO1.3
- net U1_D8: now also PIR1.1; no longer PIEZO1.1
- net U1_D9: now also R4.1, R5.1; no longer PIR1.1
- net U1_GND: now also D1.2, D2.2, R2.2; no longer GAS1.2, K1.5, K2.8, PING1.1, R1.2, R3.2, SERVO1.1
Other:
- board size 244.9 x 102.4 mm -> 139.7 x 94.2 mm
